File: cat-pcb.kicad_pcb (KiCad board)
At the start: 2 copper layers, 45 x 46.5 mm, 6 parts

Commit message: Add files via upload
Parts:
- moved D1 17.7 mm to (119.5, 81.5)
- moved D2 17.4 mm to (135.0, 81.5)
- moved R2 15.1 mm to (137.4, 85.5), turned to 0 degrees
- moved R1 14.6 mm to (116.5, 86.0), turned to 180 degrees
- moved BT1 9.12 mm to (127.0, 95.5)
- moved G*** 5.10 mm to (146.0, 73.0)
Routing:
- net Net-(BT1-+): track 54.9 -> 92.9 mm
- net Net-(BT1--): track 31.5 -> 50.5 mm
- net Net-(D2-K): track 6.54 -> 5.79 mm
- net Net-(D1-K): track 5.92 -> 6.62 mm
